Commit message: fixed gripper joint limit

File: katana_description/urdf/katana_450_6m180.urdf.xacro (robot description, xacro)
@@ -243,5 +243,5 @@
       <origin rpy="${rotate} 0 0" xyz="0.034 0 0"/>
       <axis xyz="0 0 1"/>
-      <limit effort="0.5" lower="-0.44" upper="0.30"  velocity="0.718834"/>
+      <limit effort="0.5" lower="-0.60" upper="0.30"  velocity="0.718834"/>
    </joint>
     <link name="katana_${prefix}_finger_link">

Commit message: fixed wrong rotation of gripper in urdf

File: katana_description/urdf/katana_450_6m180.urdf.xacro (robot description, xacro)
@@ -186,5 +186,5 @@
   <link name="katana_motor5_wrist_roll_link">
       <visual>
-        <origin rpy="0 ${M_PI} 0" xyz="0 0 0"/>
+        <origin rpy="0 0 0" xyz="0 0 0"/>
         <geometry>
           <mesh filename="package://katana_description/meshes/katana/katana_motor5_wrist_roll_link.stl"/>
@@ -197,5 +197,5 @@
       </visual>
       <collision>
-        <origin rpy="0 ${M_PI} 0" xyz="0 0 0"/>
+        <origin rpy="0 0 0" xyz="0 0 0"/>
         <geometry>
           <mesh filename="package://katana_description/meshes/katana/convex/katana_motor5_wrist_roll_link_convex.stl"/>
